Commit message: update

File: src/urdfs/urdf/roomba.urdf.xacro (robot description, xacro)
@@ -2,4 +2,11 @@
 <robot name="roomba" xmlns:xacro="https://www.ros.org/wiki/xacro">
     <xacro:arg name="controllers_config_path" default="" />
+    <!-- use_sim=true (default) keeps existing Gazebo behavior unchanged.
+         use_sim=false switches ros2_hardwareinterface.xacro to the real
+         ESP32 hardware plugin (see roomba_hardware package); serial_port/
+         baud_rate are only used in that case. -->
+    <xacro:arg name="use_sim" default="true" />
+    <xacro:arg name="serial_port" default="/dev/ttyUSB0" />
+    <xacro:arg name="baud_rate" default="115200" />
     <xacro:include filename="materials.xacro" />
     <xacro:include filename="inertia_descriptions.xacro" />
@@ -9,4 +16,8 @@
     <xacro:include filename="gazebo_plugin.xacro" />
     <xacro:include filename="ros2_hardwareinterface.xacro" />
+    <xacro:roomba_ros2_control
+        use_sim="$(arg use_sim)"
+        serial_port="$(arg serial_port)"
+        baud_rate="$(arg baud_rate)" />
     <xacro:property name="roomba_radius" value="0.2" />
     <xacro:property name="roomba_height" value="0.1" />

File: src/urdfs/urdf/ros2_hardwareinterface.xacro (robot description, xacro)
@@ -1,18 +1,39 @@
 <?xml version="1.0"?>
 <robot name="roomba" xmlns:xacro="https://www.ros.org/wiki/xacro">
-    <ros2_control name="GazeboSystem" type="system">
-        <hardware>
-            <plugin>gz_ros2_control/GazeboSimSystem</plugin>
-        </hardware>
-        <joint name="base_right_wheel_joint">
-            <command_interface name="velocity"/>
-            <state_interface name="velocity"/>
-            <state_interface name="position"/>
-        </joint>
-        <joint name="base_left_wheel_joint">
-            <command_interface name="velocity"/>
-            <state_interface name="velocity"/>
-            <state_interface name="position"/>
-        </joint>
-    </ros2_control>
+    <!-- use_sim=true: gz_ros2_control/GazeboSimSystem (unchanged sim behavior, default).
+         use_sim=false: roomba_hardware/ESP32SystemInterface, talking to the real
+         robot's ESP32 over serial_port @ baud_rate. Same two joints/interfaces
+         either way, so the diff_drive_controller/simple_velocity_controller +
+         planner stack above ros2_control doesn't need to know which one is active. -->
+    <xacro:macro name="roomba_ros2_control" params="use_sim serial_port baud_rate">
+        <ros2_control name="RoombaSystem" type="system">
+            <xacro:if value="${use_sim}">
+                <hardware>
+                    <plugin>gz_ros2_control/GazeboSimSystem</plugin>
+                </hardware>
+            </xacro:if>
+            <xacro:unless value="${use_sim}">
+                <hardware>
+                    <plugin>roomba_hardware/ESP32SystemInterface</plugin>
+                    <param name="serial_port">${serial_port}</param>
+                    <param name="baud_rate">${baud_rate}</param>
+                    <!-- Unverified Motor A/B to left/right mapping from the firmware
+                         side: flip these two on first bring-up if the robot spins in
+                         place or drives backwards, no rebuild needed. -->
+                    <param name="left_motor_channel">A</param>
+                    <param name="right_motor_channel">B</param>
+                </hardware>
+            </xacro:unless>
+            <joint name="base_right_wheel_joint">
+                <command_interface name="velocity"/>
+                <state_interface name="velocity"/>
+                <state_interface name="position"/>
+            </joint>
+            <joint name="base_left_wheel_joint">
+                <command_interface name="velocity"/>
+                <state_interface name="velocity"/>
+                <state_interface name="position"/>
+            </joint>
+        </ros2_control>
+    </xacro:macro>
 </robot>

Commit message: update

File: src/urdfs/urdf/roomba.urdf.xacro (robot description, xacro)
@@ -22,6 +22,6 @@
     <xacro:property name="roomba_radius" value="0.2" />
     <xacro:property name="roomba_height" value="0.1" />
-    <xacro:property name="wheel_radius" value="0.05" />
-    <xacro:property name="wheel_thickness" value="0.03" />
+    <xacro:property name="wheel_radius" value="0.035" />
+    <xacro:property name="wheel_thickness" value="0.02" />
     <link name="roomba">
     </link>
@@ -81,5 +81,5 @@
         <parent link="base_link"/>
         <child link="right_wheel"/>
-        <origin xyz="${-roomba_radius/2} ${-roomba_radius/2 - wheel_thickness/2} 0" rpy="0 0 0"/>
+        <origin xyz="${-roomba_radius/2} ${-16.65 - wheel_thickness/2} 0" rpy="0 0 0"/>
         <axis xyz="0 1 0"/>
     </joint>
@@ -87,5 +87,5 @@
         <parent link="base_link"/>
         <child link="left_wheel"/>
-        <origin xyz="${-roomba_radius/2} ${roomba_radius/2 + wheel_thickness/2} 0" rpy="0 0 0"/>
+        <origin xyz="${-roomba_radius/2} ${16.65 + wheel_thickness/2} 0" rpy="0 0 0"/>
         <axis xyz="0 1 0"/>
     </joint>

Commit message: update

File: src/urdfs/urdf/roomba.urdf.xacro (robot description, xacro)
@@ -20,5 +20,5 @@
         serial_port="$(arg serial_port)"
         baud_rate="$(arg baud_rate)" />
-    <xacro:property name="roomba_radius" value="0.2" />
+    <xacro:property name="roomba_radius" value="0.1925" />
     <xacro:property name="roomba_height" value="0.1" />
     <xacro:property name="wheel_radius" value="0.035" />
@@ -81,5 +81,5 @@
         <parent link="base_link"/>
         <child link="right_wheel"/>
-        <origin xyz="${-roomba_radius/2} ${-16.65 - wheel_thickness/2} 0" rpy="0 0 0"/>
+        <origin xyz="-0.05 ${-16.65 - wheel_thickness/2} 0" rpy="0 0 0"/>
         <axis xyz="0 1 0"/>
     </joint>
@@ -87,5 +87,5 @@
         <parent link="base_link"/>
         <child link="left_wheel"/>
-        <origin xyz="${-roomba_radius/2} ${16.65 + wheel_thickness/2} 0" rpy="0 0 0"/>
+        <origin xyz="-0.05 ${16.65 + wheel_thickness/2} 0" rpy="0 0 0"/>
         <axis xyz="0 1 0"/>
     </joint>
@@ -93,5 +93,5 @@
         <parent link="base_link"/>
         <child link="caster_wheel"/>
-        <origin xyz="${roomba_radius/4} 0 ${-wheel_radius/2}" rpy="0 0 0"/>
+        <origin xyz="0.1 0 ${-wheel_radius/2}" rpy="0 0 0"/>
     </joint>
     <joint name="spine" type="fixed">
