Commit message: update

File: src/urdfs/urdf/camera.xacro (robot description, xacro)
@@ -22,5 +22,5 @@
         <parent link="base_link" />
         <child link="camera_link" />
-        <origin xyz="${(0.4 + camera_length) / 2.0} 0 ${0.1 / 2.0}" rpy="0 0 0" />
+        <origin xyz="${(0.385 + camera_length) / 2.0} 0 ${0.1 / 2.0}" rpy="0 0 0" />
     </joint>
     <link name="camera_link_optical" />

File: src/urdfs/urdf/gazebo_plugin.xacro (robot description, xacro)
@@ -11,6 +11,6 @@
             <left_joint>base_left_wheel_joint</left_joint>
             <right_joint>base_right_wheel_joint</right_joint>
-            <wheel_separation>0.23</wheel_separation>
-            <wheel_radius>0.05</wheel_radius>
+            <wheel_separation>0.333</wheel_separation>
+            <wheel_radius>0.035</wheel_radius>
             <frame_id>odom</frame_id>
             <child_frame_id>roomba</child_frame_id>

File: src/urdfs/urdf/roomba.urdf.xacro (robot description, xacro)
@@ -81,5 +81,5 @@
         <parent link="base_link"/>
         <child link="right_wheel"/>
-        <origin xyz="-0.05 ${-16.65 - wheel_thickness/2} 0" rpy="0 0 0"/>
+        <origin xyz="-0.05 -0.1665 0" rpy="0 0 0"/>
         <axis xyz="0 1 0"/>
     </joint>
@@ -87,5 +87,5 @@
         <parent link="base_link"/>
         <child link="left_wheel"/>
-        <origin xyz="-0.05 ${16.65 + wheel_thickness/2} 0" rpy="0 0 0"/>
+        <origin xyz="-0.05 0.1665 0" rpy="0 0 0"/>
         <axis xyz="0 1 0"/>
     </joint>
