Commit message: Centralize robot dimensions in shared robot_dimensions.yaml
- add program_bringup/config/robot_dimensions.yaml and urdfs dimensions.xacro
- URDFs, sensor xacros, Gazebo plugin, relay.py, a_star and launch files
  now consume the shared geometry (20x20 cm footprint, 24 cm track,
  IMU at x=-0.08 m, body top 0.20 m above wheel centre)
- add geometry consistency tests

Co-Authored-By: Claude Sonnet 5.5 <noreply@anthropic.com>
Claude-Session: https://claude.ai/code/session_01P3ViARpXQ1n5SQwBiEvqWN

File: src/urdfs/urdf/camera.xacro (robot description, xacro)
@@ -22,5 +22,5 @@
         <parent link="base_link" />
         <child link="camera_link" />
-        <origin xyz="${(0.385 + camera_length) / 2.0} 0 ${0.1 / 2.0}" rpy="0 0 0" />
+        <origin xyz="${(footprint_length + camera_length) / 2.0} 0 ${0.1 / 2.0}" rpy="0 0 0" />
     </joint>
     <link name="camera_link_optical" />

File: src/urdfs/urdf/gazebo_plugin.xacro (robot description, xacro)
@@ -11,6 +11,6 @@
             <left_joint>base_left_wheel_joint</left_joint>
             <right_joint>base_right_wheel_joint</right_joint>
-            <wheel_separation>0.333</wheel_separation>
-            <wheel_radius>0.035</wheel_radius>
+            <wheel_separation>${track_width}</wheel_separation>
+            <wheel_radius>${wheel_radius}</wheel_radius>
             <frame_id>odom</frame_id>
             <child_frame_id>roomba</child_frame_id>

File: src/urdfs/urdf/imu_sensor.xacro (robot description, xacro)
@@ -23,5 +23,5 @@
         <parent link="base_link" />
         <child link="imu_link" />
-        <origin xyz="0 0 ${0.1 + (imu_height)}" rpy="0 0 0" />
+        <origin xyz="${imu_x} ${imu_y} ${imu_z}" rpy="0 0 0" />
     </joint>
     <gazebo reference="imu_link">

File: src/urdfs/urdf/lidar.xacro (robot description, xacro)
@@ -22,5 +22,5 @@
         <parent link="base_link" />
         <child link="lidar_link" />
-        <origin xyz="0 0 ${0.1 + (lidar_height) / 2.0}" rpy="0 0 0" />
+        <origin xyz="0 0 ${body_top_z + lidar_height / 2.0}" rpy="0 0 0" />
     </joint>
     <link name="lidar_link_optical"/>

File: src/urdfs/urdf/roomba.urdf.xacro (robot description, xacro)
@@ -9,4 +9,5 @@
     <xacro:arg name="serial_port" default="/dev/roomba_esp32" />
     <xacro:arg name="baud_rate" default="115200" />
+    <xacro:include filename="dimensions.xacro" />
     <xacro:include filename="materials.xacro" />
     <xacro:include filename="inertia_descriptions.xacro" />
@@ -20,8 +21,6 @@
         serial_port="$(arg serial_port)"
         baud_rate="$(arg baud_rate)" />
-    <xacro:property name="roomba_radius" value="0.1925" />
-    <xacro:property name="roomba_height" value="0.1" />
-    <xacro:property name="wheel_radius" value="0.035" />
-    <xacro:property name="wheel_thickness" value="0.02" />
+    <!-- footprint / wheel / caster / body dimensions: see dimensions.xacro
+         (generated from program_bringup/config/robot_dimensions.yaml) -->
     <link name="roomba">
     </link>
@@ -29,16 +28,16 @@
         <visual>
             <geometry>
-                <cylinder radius="${roomba_radius}" length="${roomba_height}" />
+                <box size="${footprint_length} ${footprint_width} ${body_height}" />
             </geometry>
-            <origin xyz="0 0 ${wheel_radius}" rpy="0 0 0" />
+            <origin xyz="0 0 ${body_center_z}" rpy="0 0 0" />
             <material name="blue" />
         </visual>
         <collision>
             <geometry>
-                <cylinder radius="${roomba_radius}" length="${roomba_height}" />
+                <box size="${footprint_length} ${footprint_width} ${body_height}" />
             </geometry>
-            <origin xyz="0 0 ${wheel_radius}" rpy="0 0 0" />
+            <origin xyz="0 0 ${body_center_z}" rpy="0 0 0" />
         </collision>
-        <xacro:cylinder_inertia Mass="10.0" r="${roomba_radius}" h="${roomba_height}" arr_xyz="0 0 ${wheel_radius}" arr_rpy="0 0 0" />
+        <xacro:box_inertia Mass="10.0" x="${footprint_length}" y="${footprint_width}" z="${body_height}" arr_xyz="0 0 ${body_center_z}" arr_rpy="0 0 0" />
     </link>
     <xacro:macro name="wheel" params="params">
@@ -65,5 +64,5 @@
         <visual>
             <geometry>
-                <sphere radius="0.01755"/>
+                <sphere radius="${caster_radius}"/>
             </geometry>
             <origin xyz="0 0 0" rpy="0 0 0"/>
@@ -72,14 +71,14 @@
         <collision>
             <geometry>
-                <sphere radius="0.01755"/>
+                <sphere radius="${caster_radius}"/>
             </geometry>
             <origin xyz="0 0 0" rpy="0 0 0"/>
         </collision>
-        <xacro:solid_sphere_inertia Mass="0.5" r="0.01755" arr_xyz="0 0 0" arr_rpy="0 0 0"/>
+        <xacro:solid_sphere_inertia Mass="0.5" r="${caster_radius}" arr_xyz="0 0 0" arr_rpy="0 0 0"/>
     </link>
     <joint name="base_right_wheel_joint" type="continuous">
         <parent link="base_link"/>
         <child link="right_wheel"/>
-        <origin xyz="-0.05 -0.1665 0" rpy="0 0 0"/>
+        <origin xyz="${wheel_axle_x} ${-track_width / 2.0} 0" rpy="0 0 0"/>
         <axis xyz="0 1 0"/>
     </joint>
@@ -87,5 +86,5 @@
         <parent link="base_link"/>
         <child link="left_wheel"/>
-        <origin xyz="-0.05 0.1665 0" rpy="0 0 0"/>
+        <origin xyz="${wheel_axle_x} ${track_width / 2.0} 0" rpy="0 0 0"/>
         <axis xyz="0 1 0"/>
     </joint>
@@ -93,5 +92,5 @@
         <parent link="base_link"/>
         <child link="caster_wheel"/>
-        <origin xyz="0.1 0 ${-wheel_radius/2}" rpy="0 0 0"/>
+        <origin xyz="${caster_x} 0 ${caster_z}" rpy="0 0 0"/>
     </joint>
     <joint name="spine" type="fixed">

File: src/urdfs/urdf/roomba_hardware.urdf.xacro (robot description, xacro)
@@ -9,4 +9,5 @@
     <xacro:arg name="serial_port" default="/dev/roomba_esp32" />
     <xacro:arg name="baud_rate" default="115200" />
+    <xacro:include filename="dimensions.xacro" />
     <xacro:include filename="materials.xacro" />
     <xacro:include filename="inertia_descriptions.xacro" />
@@ -16,8 +17,6 @@
         serial_port="$(arg serial_port)"
         baud_rate="$(arg baud_rate)" />
-    <xacro:property name="roomba_radius" value="0.1925" />
-    <xacro:property name="roomba_height" value="0.1" />
-    <xacro:property name="wheel_radius" value="0.035" />
-    <xacro:property name="wheel_thickness" value="0.02" />
+    <!-- footprint / wheel / caster / body dimensions: see dimensions.xacro
+         (generated from program_bringup/config/robot_dimensions.yaml) -->
     <link name="roomba">
     </link>
@@ -25,16 +24,16 @@
         <visual>
             <geometry>
-                <cylinder radius="${roomba_radius}" length="${roomba_height}" />
+                <box size="${footprint_length} ${footprint_width} ${body_height}" />
             </geometry>
-            <origin xyz="0 0 ${wheel_radius}" rpy="0 0 0" />
+            <origin xyz="0 0 ${body_center_z}" rpy="0 0 0" />
             <material name="blue" />
         </visual>
         <collision>
             <geometry>
-                <cylinder radius="${roomba_radius}" length="${roomba_height}" />
+                <box size="${footprint_length} ${footprint_width} ${body_height}" />
             </geometry>
-            <origin xyz="0 0 ${wheel_radius}" rpy="0 0 0" />
+            <origin xyz="0 0 ${body_center_z}" rpy="0 0 0" />
         </collision>
-        <xacro:cylinder_inertia Mass="10.0" r="${roomba_radius}" h="${roomba_height}" arr_xyz="0 0 ${wheel_radius}" arr_rpy="0 0 0" />
+        <xacro:box_inertia Mass="10.0" x="${footprint_length}" y="${footprint_width}" z="${body_height}" arr_xyz="0 0 ${body_center_z}" arr_rpy="0 0 0" />
     </link>
     <xacro:macro name="wheel" params="params">
@@ -61,5 +60,5 @@
         <visual>
             <geometry>
-                <sphere radius="0.01755"/>
+                <sphere radius="${caster_radius}"/>
             </geometry>
             <origin xyz="0 0 0" rpy="0 0 0"/>
@@ -68,14 +67,14 @@
         <collision>
             <geometry>
-                <sphere radius="0.01755"/>
+                <sphere radius="${caster_radius}"/>
             </geometry>
             <origin xyz="0 0 0" rpy="0 0 0"/>
         </collision>
-        <xacro:solid_sphere_inertia Mass="0.5" r="0.01755" arr_xyz="0 0 0" arr_rpy="0 0 0"/>
+        <xacro:solid_sphere_inertia Mass="0.5" r="${caster_radius}" arr_xyz="0 0 0" arr_rpy="0 0 0"/>
     </link>
     <joint name="base_right_wheel_joint" type="continuous">
         <parent link="base_link"/>
         <child link="right_wheel"/>
-        <origin xyz="-0.05 -0.1665 0" rpy="0 0 0"/>
+        <origin xyz="${wheel_axle_x} ${-track_width / 2.0} 0" rpy="0 0 0"/>
         <axis xyz="0 1 0"/>
     </joint>
@@ -83,5 +82,5 @@
         <parent link="base_link"/>
         <child link="left_wheel"/>
-        <origin xyz="-0.05 0.1665 0" rpy="0 0 0"/>
+        <origin xyz="${wheel_axle_x} ${track_width / 2.0} 0" rpy="0 0 0"/>
         <axis xyz="0 1 0"/>
     </joint>
@@ -89,5 +88,5 @@
         <parent link="base_link"/>
         <child link="caster_wheel"/>
-        <origin xyz="0.1 0 ${-wheel_radius/2}" rpy="0 0 0"/>
+        <origin xyz="${caster_x} 0 ${caster_z}" rpy="0 0 0"/>
     </joint>
     <joint name="spine" type="fixed">
@@ -117,5 +116,5 @@
         <parent link="base_link" />
         <child link="lidar_link" />
-        <origin xyz="0.1 0 ${0.1 + (lidar_height) / 2.0}" rpy="0 0 0" />
+        <origin xyz="${lidar_x} 0 ${body_top_z + lidar_height / 2.0}" rpy="0 0 0" />
     </joint>
     <link name="lidar_link_optical"/>
@@ -147,5 +146,5 @@
         <parent link="base_link" />
         <child link="imu_link" />
-        <origin xyz="0 0 ${0.1 + (imu_height)}" rpy="0 0 0" />
+        <origin xyz="${imu_x} ${imu_y} ${imu_z}" rpy="0 0 0" />
     </joint>
 </robot>
