Commit message: update

File: src/urdfs/urdf/gazebo_plugin.xacro (robot description, xacro)
@@ -5,5 +5,5 @@
         <mu2 value="0.01" />
     </gazebo>
-    <gazebo>
+    <!-- <gazebo>
         <plugin
             filename="gz-sim-diff-drive-system"
@@ -16,5 +16,5 @@
             <child_frame_id>roomba</child_frame_id>
         </plugin>
-    </gazebo>
+    </gazebo> -->
     <gazebo>
         <plugin

File: src/urdfs/urdf/roomba.urdf.xacro (robot description, xacro)
@@ -65,5 +65,5 @@
         <visual>
             <geometry>
-                <sphere radius="0.025"/>
+                <sphere radius="0.01755"/>
             </geometry>
             <origin xyz="0 0 0" rpy="0 0 0"/>
@@ -72,9 +72,9 @@
         <collision>
             <geometry>
-                <sphere radius="0.025"/>
+                <sphere radius="0.01755"/>
             </geometry>
             <origin xyz="0 0 0" rpy="0 0 0"/>
         </collision>
-        <xacro:solid_sphere_inertia Mass="0.5" r="0.025" arr_xyz="0 0 0" arr_rpy="0 0 0"/>
+        <xacro:solid_sphere_inertia Mass="0.5" r="0.01755" arr_xyz="0 0 0" arr_rpy="0 0 0"/>
     </link>
     <joint name="base_right_wheel_joint" type="continuous">
