Commit message: update

File: src/urdfs/urdf/roomba_hardware.urdf.xacro (robot description, xacro)
@@ -117,5 +117,5 @@
         <parent link="base_link" />
         <child link="lidar_link" />
-        <origin xyz="0 0 ${0.1 + (lidar_height) / 2.0}" rpy="0 0 0" />
+        <origin xyz="0.1 0 ${0.1 + (lidar_height) / 2.0}" rpy="0 0 0" />
     </joint>
     <link name="lidar_link_optical"/>

Commit message: update

File: src/urdfs/urdf/roomba_hardware.urdf.xacro (robot description, xacro)
@@ -110,5 +110,5 @@
         <parent link="base_link" />
         <child link="lidar_link" />
-        <origin xyz="${lidar_x} 0 ${body_top_z + lidar_height / 2.0}" rpy="0 0 0" />
+        <origin xyz="0 0 ${body_top_z + lidar_height / 2.0}" rpy="0 0 0" />
     </joint>
     <link name="lidar_link_optical"/>
